File: PCB/PJS.sch (KiCad schematic (older format))
At the start: 40 parts, among them J1 HFW8R-1STE1H1LF_FFC, K1 G2R-2-DC5_Relay, Q1 MMBT222A_Transistor, X1 XT30-F_MotorConnector, X2 XT30-F_MotorConnector, X3 XT60-F_BatteryConnector

Commit message: Jumper Connector
Parts:
- added X4: XT60-F_BatteryJumperSwitch, PJS:XT60_FemaleBatteryConnector, symbol PJS:XT60-F_BatteryJumperSwitch
Connections:
- net +12V: now also X4.2 (GND); no longer X3.1 (VOUT)
- new net: X3.1 (VOUT), X4.1 (VOUT)
Other:
- moved on the sheet: VR1

Commit message: Replacement files
Parts:
- removed A7: Teensy4.0, PJS:Teensy4.0, symbol PJS-rescue:Teensy4.0-PJS
- removed S1, S2, S3, S4: JST_2Pin, PJS:JST_2Pin, symbol PJS:JST_2Pin
- removed S5, S6, S7, S8, S9: JST_2Pin, symbol PJS:JST_2Pin
- removed X4: XT60-F_BatteryJumperSwitch, PJS:XT60_FemaleBatteryConnector, symbol PJS:XT60-F_BatteryJumperSwitch
- added J10, J6, J7, J8, J9: SM02B-PASS-TBT_SwitchConnector, PJS:SM02B-PASS-TBT_SwitchConnector, symbol PJS:SM02B-PASS-TBT_SwitchConnector
- added J2, J3, J4, J5: B02P-VL_MotorConnector, PJS:B02P-VL_MotorConnector, symbol PJS:B02P-VL_MotorConnector
- added U2: Teensy4.0, PJS:Teensy4.0, symbol PJS:Teensy4.0
- added X4: XT60-F_BatteryConnector, PJS:XT60_FemaleBatteryConnector, symbol PJS:XT60-F_BatteryConnector
- K1: footprint PJS:G2R-2-DC5 -> PJS:G2R-2-DC5_Relay
- R5: footprint PJS:MicroSD_Slot -> PJS:RMCF2512FT2K00_Resistor
- gave numbers to parts that had none: 1
Connections:
- net +12V: now also X4.2 (GND)
- net +5V: now also U2.T_VIN (VIN)
- net 3.3V_Coin: now also U2.VBAT
- net Alt_SCK: now also U2.19 (19_A5_SCL0)
- net Alt_SDI: now also U2.18 (18_A4_SDA0)
- net GND: now also J10.2 (InB), J6.2 (InB), J7.2 (InB), J8.2 (InB), J9.2 (InB), U2.G1 (GND), U2.GND, U2.~ (VUSB)
- net Link_DriverInA: now also U2.15 (15_A1_RX3_SPDIF_IN)
- net Link_DriverInB: now also U2.16 (16_A2_RX4_SCL1)
- net Link_DriverOutA: now also J3.1 (InA)
- net Link_DriverOutB: now also J3.2 (InB)
- net Link_DriverPWM: now also U2.14 (14_A0_TX3_SPDIF_OUT)
- net LockA_DriverOUT1: now also J4.1 (InA)
- net LockA_DriverOut2: now also J4.2 (InB)
- net LockB_DriverOUT1: now also J5.1 (InA)
- net LockB_DriverOUT2: now also J5.2 (InB)
- net RF_CH1: now also U2.6 (6_OUT1D)
- net RF_CH2: now also U2.7 (7_RX2_OUT1A)
- net RF_CH3: now also U2.8 (8_TX2_IN1)
- net RF_CH4: now also U2.9 (9_OUT1C)
- net Relay_Signal: now also U2.23 (23_A9_CRX1_MCLK1)
- net S1_Link: now also J6.1 (InA), J7.1 (InA), U2.2 (2_OUT2)
- net S2_Door: now also J8.1 (InA), J9.1 (InA), U2.3 (3_LRCLK2)
- net S3_UAS: now also J10.1 (InA), U2.1 (1_TX1_CTX2_MISO1)
- net SD_CLK: now also U2.36 (36_CLK_CS2)
- net SD_CMD: now also U2.37 (37_CMD_SCK2)
- net SD_DAT0: now also U2.35 (35_DAT0_MOSI2)
- net SD_DAT1: now also U2.34 (34_DAT1_MISO2)
- net SD_DAT2: now also U2.39 (39_DAT2_TX5)
- net SD_DAT3: now also U2.38 (38_DAT3_RX5)
- net SD_VDD: now also U2.~ (VUSB)
- net UAS_DriverIN1: now also U2.4 (4_BCLK2)
- net UAS_DriverIN2: now also U2.5 (5_IN2)
- net UAS_DriverOUT1: now also J2.1 (InA)
- net UAS_DriverOUT2: now also J2.2 (InB)
- net at X3.1 (VOUT): now also X4.1 (VOUT)
Other:
- moved on the sheet: U1, VR1
