File: UAS_Teensy_PCB/UAS_Teensy/UAS_Teensy.kicad_pcb (KiCad board)
At the start: 2 copper layers, 50.8 x 50.8 mm, 10 parts, among them J1 UAS-rescue_SM02B-PASS-TBT(LF)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, J2 SM04B-GHS-TB(LF)(SN)-, J3 SM07B-GHS-TB(LF)(SN), J4 SM07B-GHS-TB(LF)(SN), J5 SM04B-GHS-TB(LF)(SN)-, J6 SM04B-GHS-TB(LF)(SN)-, J7 SM04B-GHS-TB(LF)(SN)-, U1 Teensy4.0, U2 BNO055

Commit message: For Realsies Final Teensy PCB
lol
Parts:
- added J8: UAS-rescue_SM02B-PASS-TBT(LF)(SN)-SM02B-PASS-TBT_LF__SN_, UAS_Teensy:SM02BGHSTBLFSN, F.Cu at (81.3, 94.5)
Routing:
- net 5V: track 116.5 -> 136.2 mm
- net Net-(J5-Pad2): track 30.1 -> 35.7 mm
- net GND: track 12.2 -> 17.7 mm, vias 9 -> 13
- net Net-(J5-Pad1): track 34.2 -> 39.7 mm

Commit message: final version
Parts:
- added U3: Test_Pad, UAS_Teensy:Individual_Solder_Pad, F.Cu at (84.6, 101.1)
- added U4: Test_Pad, UAS_Teensy:Individual_Solder_Pad, F.Cu at (121.7, 101.1)
Connections:
- J8 pad 1: GND -> 5V
- J8 pad 2: 5V -> GND
Routing:
- net GND: track 17.7 -> 23.9 mm
- net 5V: track 136.2 -> 138.6 mm, vias 4 -> 3
- net Net-(J5-Pad2): track 35.7 -> 33.8 mm
- net Net-(J5-Pad1): track 39.7 -> 38.2 mm, vias 0 -> 1
Other:
- board text added: "Created By: Rani "Based God" Hanna"
- board text added: "JLCJLCJLCJLC"
- board text added: "rani don't touch"

Commit message: UAS PDP PCB Models
Routing:
- net (no net): vias 0 -> 4
Other:
- outline, holes or cut-outs redrawn
Changed lines of the file:
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@@
   (general
     (thickness 1.6)
-    (drawings 21472)
-    (tracks 208)
+    (drawings 21468)
+    (tracks 212)
     (zones 0)
     (modules 13)
@@
   )
   (setup
-    (last_trace_width 0.5)
+    (last_trace_width 0.127)
     (user_trace_width 0.15)
     (user_trace_width 0.2)
@@
     (user_via 1.7 1.4)
     (user_via 1.9 1.6)
+    (user_via 2.25 2)
     (uvia_size 0.6)
     (uvia_drill 0.3)
@@
     (visible_elements 7FFFFFFF)
     (pcbplotparams
-      (layerselection 0x00030_80000001)
-      (usegerberextensions false)
+      (layerselection 0x010fc_ffffffff)
+      (usegerberextensions true)
       (usegerberattributes false)
       (usegerberadvancedattributes false)
       (creategerberjobfile false)
       (excludeedgelayer true)
-      (linewidth 0.100000)
+      (linewidth 0.150000)
       (plotframeref false)
       (viasonmask false)
@@
       (psa4output false)
       (plotreference true)
-      (plotvalue true)
+      (plotvalue false)
       (plotinvisibletext false)
       (padsonsilk false)
-      (subtractmaskfromsilk false)
+      (subtractmaskfromsilk true)
       (outputformat 1)
       (mirror false)
-      (drillshape 1)
+      (drillshape 0)
       (scaleselection 1)
-      (outputdirectory ""))
+      (outputdirectory "gerbers/attempt2/"))
   )
   (net 0 "")
@@
   (gr_line (start 127 104.139999) (end 81.280001 104.139999) (layer Edge.Cuts) (width 0.05))
   (gr_arc (start 128.27 78.4225) (end 129.54 78.4225) (angle -90) (layer Edge.Cuts) (width 0.05))
-  (gr_circle (center 86.36 55.88) (end 87.63 55.88) (layer Edge.Cuts) (width 0.05))
   (gr_arc (start 86.36 55.88) (end 86.36 53.34) (angle -90) (layer Edge.Cuts) (width 0.05))
-  (gr_circle (center 127 101.6) (end 128.27 101.6) (layer Edge.Cuts) (width 0.05))
   (gr_line (start 124.46 55.88) (end 124.46 77.1525) (layer Edge.Cuts) (width 0.05))
   (gr_line (start 78.740001 101.6) (end 78.740001 78.4225) (layer Edge.Cuts) (width 0.05))
-  (gr_circle (center 81.280001 101.6) (end 82.550001 101.6) (layer Edge.Cuts) (width 0.05))
-  (gr_circle (center 121.92 55.88) (end 123.19 55.88) (layer Edge.Cuts) (width 0.05))
   (gr_arc (start 121.92 55.88) (end 124.46 55.88) (angle -90) (layer Edge.Cuts) (width 0.05))
   (gr_line (start 80.010001 77.1525) (end 83.82 77.1525) (layer Edge.Cuts) (width 0.05))
@@
   (gr_line (start 86.36 53.34) (end 121.92 53.34) (layer Edge.Cuts) (width 0.05))
   (gr_arc (start 127 101.6) (end 127 104.139999) (angle -90) (layer Edge.Cuts) (width 0.05))
+  (via (at 86.36 55.88) (size 2.25) (drill 2) (layers F.Cu B.Cu) (net 0))
+  (via (at 121.92 55.88) (size 2.25) (drill 2) (layers F.Cu B.Cu) (net 0))
+  (via (at 127 101.6) (size 2.25) (drill 2) (layers F.Cu B.Cu) (net 0))
+  (via (at 81.28 101.6) (size 2.25) (drill 2) (layers F.Cu B.Cu) (net 0))
   (segment (start 102.87 95.631) (end 102.87 95.25) (width 0.127) (layer F.Cu) (net 1))
   (segment (start 101.727 96.774) (end 102.87 95.631) (width 0.2) (layer F.Cu) (net 1))
